File: SX1255 RPI4-5 HAT.kicad_sch (KiCad schematic)
At the start: 53 parts, among them IC1 SX1255, J1 TX_SMA, J2 RX_SMA, J3 RPi, U1 MCP1703Ax-330xxMB, U3 TQP3M9036, Y1 36.864MHz / 38.40MHz

Commit message: Add files via upload
Other:
- note added: "for KDS osc. DSA321SDN (VC-TCXO) > R12 deattached, RV1-R13-R14 attached DSB321SDN (TCXO) > R12 attached, RV1-R13-R14 deattached"
Changed lines of the file:
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@@
+		)
+	)
+	(text "for KDS osc.\nDSA321SDN (VC-TCXO) > R12 deattached, RV1-R13-R14 attached\nDSB321SDN (TCXO) > R12 attached, RV1-R13-R14 deattached"
+		(exclude_from_sim no)
+		(at 33.782 82.042 0)
+		(effects
+			(font
+				(size 0.7 0.7)
+			)
 		)
 	)
