File: SX1255 RPI4-5 HAT.kicad_pcb (KiCad board)
At the start: 2 copper layers, 65 x 56.2 mm, 53 parts, among them IC1 SX1255, J1 TX_SMA, J2 RX_SMA, J3 RPi, U1 MCP1703Ax-330xxMB, U3 TQP3M9036, Y1 36.864MHz / 38.40MHz

Commit message: Add files via upload
Parts:
- removed R17: 33K, Resistor_SMD:R_0805_2012Metric
- removed R18: 10K, Resistor_SMD:R_0805_2012Metric
- removed TP: v-ref, TestPoint:TestPoint_Pad_D1.0mm
- added TP1: +5V, TestPoint:TestPoint_Pad_D1.0mm, F.Cu at (143.8, 115.5)
- added TP2: +3V3, TestPoint:TestPoint_Pad_D1.0mm, F.Cu at (145.5, 99.8)
- added TP3: OCS, TestPoint:TestPoint_Pad_D1.0mm, F.Cu at (141.5, 89.2)
- added TP4: Vcont., TestPoint:TestPoint_Pad_D1.0mm, F.Cu at (155.5, 82.2)
- moved FL1 8.75 mm to (153.0, 105.7)
- moved C31 4.51 mm to (148.2, 113.0), turned to 180 degrees
- moved C28 4.47 mm to (149.2, 106.5), turned to 90 degrees
- moved U3 1.50 mm to (144.5, 107.6)
- moved L4 1.25 mm to (149.2, 110.2)
- moved C30 0.90 mm to (148.2, 115.0)
Connections:
- U3 pad 6: /S_D -> unconnected-(U3-Pad6)
Routing:
- net /S_D: track 9.43 -> 0.00 mm, vias 2 -> 0
- net /RF-out: track 9.12 -> 5.52 mm
- net Net-(FL1-IN): track 4.71 -> 2.18 mm
- net +3V3: track 98.4 -> 96.6 mm
- net Net-(FL1-OUT): track 7.04 -> 5.33 mm
- net Net-(C11-Pad2): track 4.85 -> 3.35 mm
- net /SD: track 1.50 -> 0.00 mm
- net GND: vias 27 -> 78
- net (no net): vias 1 -> 0
