File: SX1255 RPI4-5 HAT.kicad_pcb (KiCad board)
At the start: 2 copper layers, 65 x 56.2 mm, 54 parts, among them IC1 SX1255, J1 TX_SMA, J2 RX_SMA, J3 RPi, U1 MCP1703Ax-330xxMB, U3 TQP3M9036, Y1 36.864MHz / 38.40MHz

Commit message: Add files via upload
Parts:
- added REF**: OSHW-Logo_5.7x6mm_SilkScreen, Symbol:OSHW-Logo_5.7x6mm_SilkScreen, F.Cu at (115.2, 112.2)
Other:
- board text added: "V2.2"
- board text added: "Z32IT"
